File: kicad_proj/cholatte.kicad_pcb (KiCad board)
At the start: 2 copper layers, 24 parts

Commit message: v0.1 kicad pcb
Parts:
- added D1: , ComboDiode, F.Cu at (-8.25, 0.00)
- added D10: , ComboDiode, F.Cu at (48.8, -9.00)
- added D11: , ComboDiode, F.Cu at (48.8, -26.0)
- added D12: , ComboDiode, F.Cu at (48.8, -43.0)
- added D13: , ComboDiode, F.Cu at (67.8, -7.00)
- added D14: , ComboDiode, F.Cu at (67.8, -24.0)
- added D15: , ComboDiode, F.Cu at (67.8, -41.0)
- added D16: , ComboDiode, F.Cu at (86.8, -5.00)
- added D17: , ComboDiode, F.Cu at (86.8, -22.0)
- added D18: , ComboDiode, F.Cu at (86.8, -39.0)
- added D19: , ComboDiode, F.Cu at (61.8, 15.0)
- added D2: , ComboDiode, F.Cu at (-8.25, -17.0)
- added D20: , ComboDiode, F.Cu at (84.2, 16.2)
- added D21: , ComboDiode, F.Cu at (105.0, 25.0)
- added D3: , ComboDiode, F.Cu at (-8.25, -34.0)
- added D4: , ComboDiode, F.Cu at (10.8, -2.00)
- added D5: , ComboDiode, F.Cu at (10.8, -19.0)
- added D6: , ComboDiode, F.Cu at (10.8, -36.0)
- added D7: , ComboDiode, F.Cu at (29.8, -6.00)
- added D8: , ComboDiode, F.Cu at (29.8, -23.0)
- added D9: , ComboDiode, F.Cu at (29.8, -40.0)
- added LED1: , WS2812B, F.Cu at (0.00, 5.00)
- added LED10: , WS2812B, F.Cu at (57.0, -4.00)
- added LED11: , WS2812B, F.Cu at (57.0, -21.0)
- added LED12: , WS2812B, F.Cu at (57.0, -38.0)
- added LED13: , WS2812B, F.Cu at (76.0, -2.00)
- added LED14: , WS2812B, F.Cu at (76.0, -19.0)
- added LED15: , WS2812B, F.Cu at (76.0, -36.0)
- added LED16: , WS2812B, F.Cu at (95.0, 0.00)
- added LED17: , WS2812B, F.Cu at (95.0, -17.0)
- added LED18: , WS2812B, F.Cu at (95.0, -34.0)
- added LED19: , WS2812B, F.Cu at (70.0, 20.0)
- added LED2: , WS2812B, F.Cu at (0.00, -12.0)
- added LED20: , WS2812B, F.Cu at (90.3, 23.7)
- added LED21: , WS2812B, F.Cu at (108.1, 34.1)
- added LED3: , WS2812B, F.Cu at (0.00, -29.0)
- added LED4: , WS2812B, F.Cu at (19.0, 3.00)
- added LED5: , WS2812B, F.Cu at (19.0, -14.0)
- added LED6: , WS2812B, F.Cu at (19.0, -31.0)
- added LED7: , WS2812B, F.Cu at (38.0, -1.00)
- added LED8: , WS2812B, F.Cu at (38.0, -18.0)
- added LED9: , WS2812B, F.Cu at (38.0, -35.0)
- moved REF** 5.00 mm to (127.0, -13.0)
- moved MCU1 3.64 mm to (115.0, -37.5)
Connections:
- net matrix_thumbfan_far renamed P21
- net matrix_thumbfan_home renamed P20
- net matrix_thumbfan_near renamed P19
- MCU1 pad 10: matrix_index_home -> P14
- MCU1 pad 11: matrix_inner_bottom -> P16
- MCU1 pad 12: matrix_middle_bottom -> P10
- MCU1 pad 13: matrix_outer_bottom -> P1
- MCU1 pad 17: matrix_outer_home -> P2
- MCU1 pad 18: matrix_outer_top -> P3
- MCU1 pad 19: matrix_pinky_bottom -> P4
- MCU1 pad 20: matrix_pinky_home -> P5
- MCU1 pad 21: matrix_pinky_top -> P6
- MCU1 pad 22: matrix_ring_bottom -> P7
- MCU1 pad 23: matrix_ring_home -> P8
- MCU1 pad 24: matrix_ring_top -> P9
- MCU1 pad 8: matrix_inner_top -> P18
- MCU1 pad 9: matrix_index_top -> P15
Other:
- board outline added: 140.2 x 102.2 mm

Commit message: v0.1 ready for testing 3d printing and layout check
Parts:
- moved S21 193.5 mm to (228.5, 184.3)
- moved D20 193.5 mm to (201.5, 170.2)
- moved LED21 193.5 mm to (225.3, 188.1)
- moved D19 193.5 mm to (179.0, 169.0)
- moved LED19 193.5 mm to (187.2, 174.0)
- moved S19 193.5 mm to (187.2, 169.0)
- moved S20 193.5 mm to (209.2, 173.0)
- moved D21 193.5 mm to (222.2, 179.0)
- moved LED20 193.5 mm to (207.5, 177.7)
- moved D1 189.4 mm to (102.0, 154.0)
- moved D10 189.4 mm to (159.0, 145.0)
- moved D13 189.4 mm to (178.0, 147.0)
- moved D16 189.4 mm to (197.0, 149.0)
- moved D4 189.4 mm to (121.0, 152.0)
- moved D7 189.4 mm to (140.0, 148.0)
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Connections:
- net P19 renamed matrix_thumbfan_near
- net P20 renamed matrix_thumbfan_home
- net P21 renamed matrix_thumbfan_far
- D1 pad 1: matrix_outer_bottom -> unknown
- D1 pad 2: unknown -> matrix_outer_bottom
- D10 pad 1: matrix_middle_bottom -> unknown
- D11 pad 1: matrix_middle_home -> unknown
- D12 pad 1: matrix_middle_top -> unknown
- D12 pad 2: unknown -> matrix_middle_top
- D14 pad 1: matrix_index_home -> unknown
- D14 pad 2: unknown -> matrix_index_home
- D15 pad 2: unknown -> matrix_index_top
- D16 pad 1: matrix_inner_bottom -> unknown
- D16 pad 2: unknown -> matrix_inner_bottom
- D17 pad 1: matrix_inner_home -> unknown
- D18 pad 1: matrix_inner_top -> unknown
- D19 pad 1: thumbfan_near_thumb -> unknown
- D19 pad 2: unknown -> thumbfan_near_thumb
- D2 pad 1: matrix_outer_home -> unknown
- D20 pad 1: thumbfan_home_thumb -> unknown
- D21 pad 1: thumbfan_far_thumb -> unknown
- D3 pad 1: matrix_outer_top -> unknown
- D3 pad 2: unknown -> matrix_outer_top
- D4 pad 2: unknown -> matrix_pinky_bottom
- D5 pad 1: matrix_pinky_home -> unknown
- D5 pad 2: unknown -> matrix_pinky_home
- D6 pad 1: matrix_pinky_top -> unknown
- D6 pad 2: unknown -> matrix_pinky_top
- D7 pad 2: unknown -> matrix_ring_bottom
- D8 pad 1: matrix_ring_home -> unknown
- D8 pad 2: unknown -> matrix_ring_home
- MCU1 pad 10: P14 -> matrix_index_home
- MCU1 pad 11: P16 -> matrix_inner_bottom
- MCU1 pad 12: P10 -> matrix_middle_bottom
- MCU1 pad 13: P1 -> matrix_outer_bottom
- MCU1 pad 17: P2 -> matrix_outer_home
- MCU1 pad 18: P3 -> matrix_outer_top
- MCU1 pad 19: P4 -> matrix_pinky_bottom
- MCU1 pad 20: P5 -> matrix_pinky_home
- MCU1 pad 21: P6 -> matrix_pinky_top
- MCU1 pad 22: P7 -> matrix_ring_bottom
- MCU1 pad 23: P8 -> matrix_ring_home
- MCU1 pad 24: P9 -> matrix_ring_top
- MCU1 pad 8: P18 -> matrix_inner_top
- MCU1 pad 9: P15 -> matrix_index_top
Other:
- board size 140.2 x 102.2 mm -> 147.2 x 104.2 mm
- net class Default removed
- net class Power removed
